File: 572pv1.brd (EAGLE design)
At the start: 142.2 x 67 mm, 46 parts, among them IC3 74141N

Commit message: .
Parts:
- removed U$2: К161ПР2, КР1534,К161,К120:238.16-1
- added DA2: КР142ЕН1Г, linear:DIL14
- added DP10, DP11, DP12, DP13, DP14, DP9: К(М)155ПР7,(54)74184, 74xx-us:DIL16
- moved DD2 202.1 mm to (26.0, -52.7), turned to 180 degrees
- moved JGND 97.5 mm to (29.2, 61.6), flipped to the bottom, turned to 90 degrees
- moved IC1 10.8 mm to (169.5, 31.8)
- renumbered D1 to VD4, D2 to VD1, D3 to VD2
Connections:
- new net N$102: DP13.5, DP14.13
- new net N$103: DP13.6, DP14.14
- new net N$17: DP13.2, DP14.10
- new net N$96: DP13.3, DP14.11
- new net N$98: DP13.4, DP14.12
- net -VCC: no longer U$2.9
- net GND: now also DP10.8, DP11.8, DP12.8, DP13.8, DP14.8, DP9.8; no longer U$2.1
- net VCC: now also DP10.16, DP11.16, DP12.16, DP13.16, DP14.16, DP9.16
Routing:
- net N$84: track 0.00 -> 45.2 mm
- net N$66: track 0.00 -> 44.4 mm
- net N$83: track 0.00 -> 40.2 mm
- net N$67: track 0.00 -> 39.8 mm
- net N$63: track 0.00 -> 34.2 mm
- net N$55: track 0.00 -> 28.6 mm
- net N$56: track 0.00 -> 28.5 mm
- net N$59: track 0.00 -> 16.3 mm
- net GND: track 57.9 -> 42.0 mm
- net N$58: track 0.00 -> 12.5 mm
- net N$68: track 0.00 -> 12.1 mm
- net N$61: track 16.3 -> 26.4 mm
- net N$60: track 0.00 -> 8.30 mm
- net N$57: track 0.00 -> 3.81 mm
- net N$87: track 59.4 -> 56.2 mm
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
Commit message: .
Parts:
- added DI1, DI2, DI3: 4030N, 40xx:DIL14
- added DIP21_1, DIP21_2: (no value), Разъёмы штырьковые 2.54мм:1X20
- added IC5: M29F400M, st-microelectronics:SO44
- added IC6: M29F400T, st-microelectronics:TSOP48
- DP1: value К(М)155ПР7,(54)74184 -> К(М)155ПР7,(54)74185; device 74xx-us:DIL16 -> 74xx-eu:DIL16
- DP2, DP3, DP4, DP5, DP6, DP7, DP8: value 74184N -> КМ155ПР7; device 74xx-us:DIL16 -> 74xx-eu:DIL16
- moved IC1 239.1 mm to (-54.6, -51.4), turned to 0 degrees
- moved DP10 224.2 mm to (-208.3, -70.5)
- moved DP11 224.2 mm to (-182.2, -85.7)
- moved DP13 224.2 mm to (-208.3, -98.4)
- moved DP12 224.2 mm to (-205.1, -86.4)
- moved DP14 224.2 mm to (-182.9, -98.4)
- moved DP9 224.2 mm to (-184.8, -70.5)
- moved IC3 153.6 mm to (-94.6, 2.54), turned to 90 degrees
- moved U$3 146.5 mm to (-99.7, -69.8), turned to 0 degrees
- moved DD2 142.2 mm to (-116.2, -51.4)
- moved JP1 8.98 mm to (43.2, 22.9)
- moved DP7 1.91 mm to (258.4, 21.6)
- moved JP4 1.80 mm to (76.2, 22.9)
- moved DP5 1.27 mm to (247.7, 21.6)
- moved DP6 1.27 mm to (247.7, 43.2)
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Connections:
- new net N$104: DI2.11, DIP21_2.12
- new net N$105: DI2.12, DIP21_1.12
- new net N$106: DI2.5, DIP21_1.11
- new net N$107: DI1.8, DIP21_1.14
- new net N$108: DI1.6, DIP21_1.15
- new net N$109: DI1.12, DIP21_1.16
- new net N$110: DI1.1, DIP21_1.17
- new net N$111: DI2.9, DIP21_1.9
- new net N$112: DI3.1, DIP21_1.8
- new net N$113: DI3.13, DIP21_1.7
- new net N$114: DI3.8, DIP21_1.6
- new net N$115: DI2.3, DIP21_2.13
- new net N$116: DI2.1, DIP21_1.13
- new net N$117: DIP21_1.1, DIP21_1.10, DIP21_1.2, DIP21_1.3, DIP21_1.4
- new net N$118: DI1.13, DI1.2, DI1.5, DI1.9, DI2.13, DI2.2, DI2.6, DI2.8, DI3.12, DI3.2, DI3.9, DIP21_1.5
- new net N$119: DI1.10, DIP21_2.14
- new net N$120: DI1.4, DIP21_2.15
- new net N$121: DI1.11, DIP21_2.16
- new net N$122: DI1.3, DIP21_2.17
- new net N$123: DI2.4, DIP21_2.11
- new net N$124: DI2.10, DIP21_2.9
- new net N$125: DI3.3, DIP21_2.8
- new net N$126: DI3.11, DIP21_2.7
- new net N$127: DI3.10, DIP21_2.6
- new net VDD: DI1.14, DI2.14, DI3.14
- new net VSS: DI1.7, DI2.7, DI3.7
- net GND: now also IC5.13, IC5.32, IC6.27, IC6.46
- net VCC: now also IC5.23, IC6.37
Routing:
- net N$118: track 0.00 -> 112.2 mm
- net N$86: track 104.1 -> 180.1 mm
- net N$85: track 0.00 -> 65.6 mm
- net N$75: track 0.00 -> 43.4 mm
- net N$90: track 125.2 -> 164.6 mm
- net N$117: track 0.00 -> 38.7 mm
- net N$87: track 56.2 -> 93.7 mm
- net N$62: track 0.00 -> 31.8 mm, vias 0 -> 2
- net N$114: track 0.00 -> 23.4 mm
- net N$110: track 0.00 -> 21.6 mm
- net N$112: track 0.00 -> 16.2 mm
- net N$116: track 0.00 -> 15.4 mm
- net N$106: track 0.00 -> 14.9 mm
- net N$108: track 0.00 -> 14.9 mm
- net N$82: track 0.00 -> 11.5 mm
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Other:
- board text added: "1"
- board text added: "20"
- board text added: "21"
- board text added: "40"
