File: 572pv1.sch (EAGLE design)
At the start: 46 parts, among them IC3 74141N

Commit message: .
Parts:
- removed D1: (no value), diode:DIODE-SOD80C
- removed U$2: К161ПР2, КР1534,К161,К120:К161ПР2
- added DA2: КР142ЕН1Г, linear:UA723N
- added DP10, DP11, DP12, DP13, DP14, DP9: К(М)155ПР7,(54)74184, 74xx-us:74184N
- added VD4: (no value), diode:DIODE-SOD80C
- renumbered D2 to VD1, D3 to VD2
Connections:
- new net N$102: DP13A.Y5, DP14A.D
- new net N$103: DP13A.Y6, DP14A.E
- new net N$17: DP13A.Y2, DP14A.A
- new net N$96: DP13A.Y3, DP14A.B
- new net N$98: DP13A.Y4, DP14A.C
- net AGND: now also VD4.A; no longer D1.A
- net N$6: now also VD4.C; no longer D1.C
Other:
- note added: "(VD3) нужен диод с agnd на 39(выход) если 39 не соединён с agnd"
- note added: "155ПР7 нужно отключать питание когда идёт счёт"
- note added: "? КР142ЕН1Г"
- note added: "VD2 минимальное падение"
Changed lines of the file:
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@@
 <parts>
 <part name="DD1" library="572" deviceset="КР572ПВ1" device="" value="КР572ПВ1А"/>
-<part name="D1" library="diode" deviceset="DIODE-" device="SOD80C"/>
-<part name="D2" library="diode" deviceset="DIODE-" device="SOD80C"/>
-<part name="D3" library="diode" deviceset="DIODE-" device="SOD80C"/>
+<part name="VD4" library="diode" deviceset="DIODE-" device="SOD80C"/>
+<part name="VD1" library="diode" deviceset="DIODE-" device="SOD80C"/>
+<part name="VD2" library="diode" deviceset="DIODE-" device="SOD80C"/>
 <part name="GND2" library="supply1v" deviceset="GND" device=""/>
 <part name="GND3" library="supply1v" deviceset="GND" device=""/>
@@
 <part name="DIP1_20" library="Разъёмы штырьковые 2.54мм" deviceset="PINHD-1X20" device=""/>
 <part name="DIP21_40" library="Разъёмы штырьковые 2.54мм" deviceset="PINHD-1X20" device=""/>
-<part name="U$2" library="КР1534,К161,К120" deviceset="К161ПР2" device=""/>
 <part name="U$3" library="КР1534,К161,К120" deviceset="К161ПР2" device=""/>
 <part name="IC3" library="74xx-us" deviceset="74*141" device="N"/>
@@
 <part name="P+1" library="supply1v" deviceset="+5V" device=""/>
 <part name="P+2" library="supply1v" deviceset="+5V" device=""/>
+<part name="DP9" library="74xx-us" deviceset="74*184" device="N" value="К(М)155ПР7,(54)74184"/>
+<part name="DP10" library="74xx-us" deviceset="74*184" device="N" value="К(М)155ПР7,(54)74184"/>
+<part name="DP11" library="74xx-us" deviceset="74*184" device="N" value="К(М)155ПР7,(54)74184"/>
+<part name="DP12" library="74xx-us" deviceset="74*184" device="N" value="К(М)155ПР7,(54)74184"/>
+<part name="DP13" library="74xx-us" deviceset="74*184" device="N" value="К(М)155ПР7,(54)74184"/>
+<part name="DP14" library="74xx-us" deviceset="74*184" device="N" value="К(М)155ПР7,(54)74184"/>
+<part name="DA2" library="linear" deviceset="*723" device="N" technology="UA" value="КР142ЕН1Г"/>
 </parts>
 <sheets>
@@
 24 на GND</text>
 <text x="34.29" y="116.84" size="1.778" layer="98" rot="MR0">IL311ANM</text>
+<text x="66.04" y="38.1" size="1.778" layer="98" rot="MR180">(VD3) нужен диод с agnd на 39(выход)
+если 39 не соединён с agnd</text>
+<text x="58.42" y="157.48" size="1.778" layer="98" rot="MR180">VD2 минимальное падение</text>
+<text x="429.26" y="134.62" size="1.778" layer="98" rot="MR180">155ПР7 нужно отключать питание когда идёт счёт</text>
+<text x="27.94" y="182.88" size="1.778" layer="98" rot="MR180">? КР142ЕН1Г</text>
 </plain>
 <instances>
@@
 <instance part="DD1" gate=".4" x="33.02" y="30.48"/>
 <instance part="DD1" gate=".2" x="25.4" y="147.32"/>
-<instance part="D1" gate="G$1" x="48.26" y="45.72" smashed="yes">
-<attribute name="NAME" x="48.26" y="41.1226" size="1.778" layer="95"/>
-<attribute name="VALUE" x="50.8" y="43.4086" size="1.778" layer="96"/>
+<instance part="VD4" gate="G$1" x="53.34" y="40.64" smashed="yes" rot="R90">
+<attribute name="NAME" x="55.88" y="41.1226" size="1.778" layer="95"/>
+<attribute name="VALUE" x="55.6514" y="43.18" size="1.778" layer="96" rot="R90"/>
 </instance>
-<instance part="D2" gate="G$1" x="48.26" y="149.86" smashed="yes">
+<instance part="VD1" gate="G$1" x="48.26" y="149.86" smashed="yes">
 <attribute name="NAME" x="45.72" y="152.8826" size="1.778" layer="95"/>
 <attribute name="VALUE" x="50.8" y="147.5486" size="1.778" layer="96"/>
 </instance>
-<instance part="D3" gate="G$1" x="53.34" y="154.94" smashed="yes" rot="R270">
+<instance part="VD2" gate="G$1" x="53.34" y="154.94" smashed="yes" rot="R270">
 <attribute name="NAME" x="48.26" y="155.4226" size="1.778" layer="95"/>
 <attribute name="VALUE" x="51.0286" y="152.4" size="1.778" layer="96" rot="R270"/>
@@
 <instance part="DIP1_20" gate="A" x="594.36" y="101.6"/>
 <instance part="DIP21_40" gate="A" x="320.04" y="91.44" rot="R180"/>
-<instance part="U$2" gate="DD" x="629.92" y="114.3"/>
 <instance part="U$3" gate="DD" x="162.56" y="162.56" smashed="yes" rot="MR180">
 <attribute name="NAME" x="159.385" y="177.165" size="1.778" layer="95" rot="MR180"/>
@@
 <instance part="JGND" gate="G$1" x="5.08" y="157.48" rot="R90"/>
 <instance part="AGND3" gate="VR1" x="43.18" y="109.22"/>
-<instance part="AGND4" gate="VR1" x="43.18" y="40.64"/>
+<instance part="AGND4" gate="VR1" x="53.34" y="30.48"/>
 <instance part="P+1" gate="1" x="38.1" y="142.24"/>
 <instance part="P+2" gate="1" x="-2.54" y="73.66" rot="R90"/>
+<instance part="DP9" gate="A" x="213.36" y="256.54"/>
+<instance part="DP10" gate="A" x="243.84" y="256.54"/>
+<instance part="DP11" gate="A" x="274.32" y="256.54"/>
+<instance part="DP12" gate="A" x="302.26" y="256.54"/>
+<instance part="DP13" gate="A" x="271.78" y="226.06"/>
+<instance part="DP14" gate="A" x="297.18" y="223.52"/>
+<instance part="DA2" gate="A" x="33.02" y="208.28"/>
 </instances>
 <busses>
@@
 <segment>
 <pinref part="DD1" gate=".2" pin="VCC15"/>
-<pinref part="D2" gate="G$1" pin="C"/>
+<pinref part="VD1" gate="G$1" pin="C"/>
 <wire x1="38.1" y1="147.32" x2="53.34" y2="147.32" width="0.1524" layer="91"/>
 <wire x1="53.34" y1="147.32" x2="53.34" y2="149.86" width="0.1524" layer="91"/>
 <wire x1="53.34" y1="149.86" x2="50.8" y2="149.86" width="0.1524" layer="91"/>
-<pinref part="D3" gate="G$1" pin="C"/>
+<pinref part="VD2" gate="G$1" pin="C"/>
 <wire x1="53.34" y1="152.4" x2="53.34" y2="149.86" width="0.1524" layer="91"/>
 <junction x="53.34" y="149.86"/>
@@
 <pinref part="DD1" gate=".4" pin="R2"/>
 <wire x1="40.64" y1="30.48" x2="43.18" y2="30.48" width="0.1524" layer="91"/>
-<wire x1="43.18" y1="30.48" x2="53.34" y2="30.48" width="0.1524" layer="91"/>
-<wire x1="53.34" y1="30.48" x2="53.34" y2="45.72" width="0.1524" layer="91"/>
 <pinref part="DD1" gate=".1" pin="I1"/>
 <wire x1="53.34" y1="45.72" x2="53.34" y2="48.26" width="0.1524" layer="91"/>
 <wire x1="53.34" y1="48.26" x2="40.64" y2="48.26" width="0.1524" layer="91"/>
-<pinref part="D1" gate="G$1" pin="C"/>
-<wire x1="50.8" y1="45.72" x2="53.34" y2="45.72" width="0.1524" layer="91"/>
+<pinref part="VD4" gate="G$1" pin="C"/>
+<wire x1="53.34" y1="43.18" x2="53.34" y2="45.72" width="0.1524" layer="91"/>
 <junction x="53.34" y="45.72"/>
 <wire x1="43.18" y1="22.86" x2="43.18" y2="30.48" width="0.1524" layer="91"/>
 <junction x="25.4" y="22.86"/>
-<junction x="43.18" y="30.48"/>
 <wire x1="53.34" y1="48.26" x2="53.34" y2="99.06" width="0.1524" layer="91"/>
 <wire x1="53.34" y1="99.06" x2="53.34" y2="127" width="0.1524" layer="91"/>
@@
 <wire x1="50.8" y1="127" x2="48.26" y2="127" width="0.1524" layer="91"/>
 <junction x="53.34" y="48.26"/>
+<wire x1="43.18" y1="22.86" x2="60.96" y2="22.86" width="0.1524" layer="91"/>
+<wire x1="60.96" y1="22.86" x2="60.96" y2="45.72" width="0.1524" layer="91"/>
+<wire x1="60.96" y1="45.72" x2="53.34" y2="45.72" width="0.1524" layer="91"/>
+<junction x="43.18" y="22.86"/>
 </segment>
 </net>
@@
 <net name="N$97" class="0">
 <segment>
-<pinref part="D3" gate="G$1" pin="A"/>
+<pinref part="VD2" gate="G$1" pin="A"/>
 <wire x1="53.34" y1="160.02" x2="53.34" y2="157.48" width="0.1524" layer="91"/>
 <pinref part="+15V" gate="G$1" pin="1"/>
@@
 <pinref part="DD1" gate=".1" pin="I2"/>
 <wire x1="40.64" y1="45.72" x2="43.18" y2="45.72" width="0.1524" layer="91"/>
-<wire x1="43.18" y1="45.72" x2="43.18" y2="43.18" width="0.1524" layer="91"/>
-<pinref part="D1" gate="G$1" pin="A"/>
-<wire x1="45.72" y1="45.72" x2="43.18" y2="45.72" width="0.1524" layer="91"/>
-<junction x="43.18" y="45.72"/>
+<pinref part="VD4" gate="G$1" pin="A"/>
 <pinref part="AGND4" gate="VR1" pin="AGND"/>
 <pinref part="DD1" gate=".1" pin="I3"/>
 <wire x1="40.64" y1="50.8" x2="43.18" y2="50.8" width="0.1524" layer="91"/>
-<wire x1="43.18" y1="50.8" x2="43.18" y2="45.72" width="0.1524" layer="91"/>
+<wire x1="53.34" y1="33.02" x2="53.34" y2="35.56" width="0.1524" layer="91"/>
+<wire x1="53.34" y1="35.56" x2="53.34" y2="38.1" width="0.1524" layer="91"/>
+<wire x1="43.18" y1="45.72" x2="45.72" y2="45.72" width="0.1524" layer="91"/>
+<wire x1="45.72" y1="45.72" x2="45.72" y2="40.64" width="0.1524" layer="91"/>
+<junction x="53.34" y="35.56"/>
+<wire x1="48.26" y1="35.56" x2="53.34" y2="35.56" width="0.1524" layer="91"/>
+<wire x1="43.18" y1="50.8" x2="48.26" y2="50.8" width="0.1524" layer="91"/>
+<wire x1="48.26" y1="50.8" x2="48.26" y2="40.64" width="0.1524" layer="91"/>
+<wire x1="48.26" y1="40.64" x2="48.26" y2="35.56" width="0.1524" layer="91"/>
+<wire x1="45.72" y1="40.64" x2="48.26" y2="40.64" width="0.1524" layer="91"/>
+<junction x="48.26" y="40.64"/>
 </segment>
 </net>
@@
 <segment>
 <pinref part="DD1" gate=".2" pin="VCC5"/>
-<pinref part="D2" gate="G$1" pin="A"/>
+<pinref part="VD1" gate="G$1" pin="A"/>
 <wire x1="38.1" y1="149.86" x2="43.18" y2="149.86" width="0.1524" layer="91"/>
 <wire x1="43.18" y1="149.86" x2="45.72" y2="149.86" width="0.1524" layer="91"/>
@@
 </segment>
 </net>
+<net name="N$17" class="0">
+<segment>
+<pinref part="DP13" gate="A" pin="Y2"/>
+<pinref part="DP14" gate="A" pin="A"/>
+</segment>
+</net>
+<net name="N$96" class="0">
+<segment>
+<pinref part="DP13" gate="A" pin="Y3"/>
+<pinref part="DP14" gate="A" pin="B"/>
+</segment>
+</net>
+<net name="N$98" class="0">
+<segment>
+<pinref part="DP13" gate="A" pin="Y4"/>
+<pinref part="DP14" gate="A" pin="C"/>
+</segment>
+</net>
+<net name="N$102" class="0">
+<segment>
+<pinref part="DP13" gate="A" pin="Y5"/>
+<pinref part="DP14" gate="A" pin="D"/>
+</segment>
+</net>
+<net name="N$103" class="0">
+<segment>
+<pinref part="DP13" gate="A" pin="Y6"/>
+<pinref part="DP14" gate="A" pin="E"/>
+</segment>
+</net>

Commit message: .
Parts:
- added DI1, DI2, DI3: 4030N, 40xx:4030N
- added DIP21_1, DIP21_2: (no value), Разъёмы штырьковые 2.54мм:PINHD-1X20
- added IC5: M29F400M, st-microelectronics:M29F400M
- added IC6: M29F400T, st-microelectronics:M29F400T
- DP1: value К(М)155ПР7,(54)74184 -> К(М)155ПР7,(54)74185; device 74xx-us:74184N -> 74xx-eu:74184N
- DP2, DP3, DP4, DP5, DP6, DP7, DP8: value 74184N -> КМ155ПР7; device 74xx-us:74184N -> 74xx-eu:74184N
Connections:
- new net N$104: DI2D.O, DIP21_2.12
- new net N$105: DI2D.I0, DIP21_1.12
- new net N$106: DI2B.I0, DIP21_1.11
- new net N$107: DI1C.I0, DIP21_1.14
- new net N$108: DI1B.I1, DIP21_1.15
- new net N$109: DI1D.I0, DIP21_1.16
- new net N$110: DI1A.I0, DIP21_1.17
- new net N$111: DI2C.I1, DIP21_1.9
- new net N$112: DI3A.I0, DIP21_1.8
- new net N$113: DI3D.I1, DIP21_1.7
- new net N$114: DI3C.I0, DIP21_1.6
- new net N$115: DI2A.O, DIP21_2.13
- new net N$116: DI2A.I0, DIP21_1.13
- new net N$117: DIP21_1.1, DIP21_1.10, DIP21_1.2, DIP21_1.3, DIP21_1.4
- new net N$118: DI1A.I1, DI1B.I0, DI1C.I1, DI1D.I1, DI2A.I1, DI2B.I1, DI2C.I0, DI2D.I1, DI3A.I1, DI3C.I1, DI3D.I0, DIP21_1.5
- new net N$119: DI1C.O, DIP21_2.14
- new net N$120: DI1B.O, DIP21_2.15
- new net N$121: DI1D.O, DIP21_2.16
- new net N$122: DI1A.O, DIP21_2.17
- new net N$123: DI2B.O, DIP21_2.11
- new net N$124: DI2C.O, DIP21_2.9
- new net N$125: DI3A.O, DIP21_2.8
- new net N$126: DI3D.O, DIP21_2.7
- new net N$127: DI3C.O, DIP21_2.6
Other:
- note added: "17. !0 АЦП!,1 ЦАП"
- note added: "24. !0 ждущий!,к22 непрерывный"
- note added: "SO44, TS48 Am29F200B 2M(256k x8 or 128k x16)"
- note added: "Деление 2^0..2^12=0..4096 до -2048 Старший разряд 1 знак +. Отсчёт = младшие разряды +1. Старший разряд 0 знак -. Другие разряды инвертировать"
- note added: "К155ПР7 матричная К155РЕ3. КМ155ПР7, в керамике РЕ3 не найдена. 74185 заказная масочная SN7488"
- note added: "Цена ПР7/РЕ3 15р.х8шт.=120р"
- note added: "перевернуть полюса микросхем"
- note added: "полярность низ младший разряд 15..8 7..4 верх старший"
- note added: "поменять полярность низ старший разряд верх младший"
- moved on the sheet: +15V, +5V, -10.24V, 01, 02, 03, 04, C1, C2, DA1, DD1.2, DIP1_20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
